Commit message: feat: smaller dae file suitable for foxglove

File: pixkit_description/urdf/vehicle.xacro (robot description, xacro)
@@ -1,4 +1,4 @@
 <?xml version="1.0"?>
-<robot xmlns:xacro="http://ros.org/wiki/xacro">
+<robot name="pixloop" xmlns:xacro="http://ros.org/wiki/xacro">
   <!-- load parameter -->
   <xacro:property name="vehicle_info" value="${xacro.load_yaml('$(find pixkit_description)/config/vehicle_info.param.yaml')}"/>
@@ -12,11 +12,3 @@
     </visual>
   </link>
-  <!-- <link name="base_link">
-    <visual>
-      <origin xyz="${vehicle_info['/**']['ros__parameters']['wheel_base']/2.0} 0 0" rpy="${pi/2.0} 0 ${pi}"/>
-      <geometry>
-        <mesh filename="package://pixkit_description/mesh/lexus.dae" scale="1 1 1"/>
-      </geometry>
-    </visual>
-  </link> -->
 </robot>
